File: electronics/generated/carrier/carrier.kicad_pcb (KiCad board)
At the start: 2 copper layers, 80 x 100 mm, 15 parts, among them J1 EXTERNAL_3V3_CURRENT_LIMITED, J2 SPI_BANK_0, J3 SPI_BANK_1, J4 SPI_BANK_2, J5 SPI_BANK_3, J6 ADXL355_3V3_MODULE, J7 ODOMETER_3V3_ONLY, U1 Raspberry_Pi_Pico_USB_powered

Commit message: build(electronics): publish KiCad, routed boards, schematics and checks [skip ci]
Routing:
- net MISO1: track 51.8 -> 59.7 mm
- net SCK0: track 84.4 -> 77.9 mm
- net GND: track 224.2 -> 229.1 mm
- net MISO0: track 85.6 -> 80.7 mm
- net MOSI1: track 58.2 -> 62.2 mm
- net SCK1: track 56.3 -> 59.1 mm
- net CS0: track 45.2 -> 47.0 mm, vias 0 -> 1
- net CS_ADXL: track 54.4 -> 52.7 mm
- net MOSI0: track 81.3 -> 80.1 mm
- net EXT_3V3: track 7.11 -> 6.58 mm

Commit message: build: publish checked electronics/generated [skip ci]
Routing:
- net MOSI1: track 62.2 -> 50.8 mm
- net MOSI0: track 80.1 -> 87.8 mm
- net MISO0: track 80.7 -> 85.6 mm
- net GND: track 229.1 -> 225.7 mm
- net MISO1: track 59.7 -> 62.2 mm
- net CS0: track 47.0 -> 45.2 mm, vias 1 -> 0
- net CS_ADXL: track 52.7 -> 54.0 mm
