File: electronics/generated/encoder/encoder.kicad_pcb (KiCad board)
At the start: 2 copper layers, 18 x 24 mm, 6 parts, among them J1 CHAIN_3V3_ONLY, U1 AS5048A

Commit message: build(electronics): publish KiCad, routed boards, schematics and checks [skip ci]
Routing:
- net CS: track 7.82 -> 8.40 mm

Commit message: build: publish checked electronics/generated [skip ci]
Routing:
- net CS: track 8.40 -> 7.82 mm
