File: electronics/generated/encoder/encoder.kicad_sch (KiCad schematic)
At the start: 4 parts, among them J1 CHAIN_3V3_ONLY, U1 AS5048A

Commit message: build: publish checked electronics/generated [skip ci]
Other:
- moved on the sheet: C1, C2, U1
