File: electronics/generated-r2/force/force.kicad_sch (KiCad schematic)
At the start: 5 parts, among them J1 HALL_3V3_GND_OUT, U1 DRV5055A3DBZR

Commit message: build(r2): publish final routed electronics and checks [skip ci]
Parts:
- U1: value DRV5055A3DBZR -> DRV5055A3QDBZR
